Commit message: Changed origin of robot

File: franka_description/robots/panda_arm.xacro (robot description, xacro)
@@ -14,5 +14,5 @@
       <parent link="world" />
       <child link="${arm_id}_link0" />
-      <origin xyz="0.0 0.0 0.0" rpy="0.0 0.0 0.0" />
+      <origin xyz="0.65 0.3 1.04" rpy="0.0 0.0 0.0" />
     </joint>
     <xacro:property name="joint_damping" value="1.0"/>

Commit message: Changed parameters of robot

File: franka_description/robots/panda_arm.xacro (robot description, xacro)
@@ -14,5 +14,5 @@
       <parent link="world" />
       <child link="${arm_id}_link0" />
-      <origin xyz="0.65 0.3 1.04" rpy="0.0 0.0 0.0" />
+      <origin xyz="0 0 0" rpy="0.0 0.0 0.0" />
     </joint>
     <xacro:property name="joint_damping" value="1.0"/>

File: franka_description/robots/panda_arm_hand_ctrl.urdf.xacro (robot description, xacro)
@@ -26,6 +26,5 @@
   <xacro:unless value="$(arg use_ros_control)">
         <xacro:include filename="$(find jaco_gazebo)/urdf/gzplugin_joint_control.urdf.xacro"/>
-        <xacro:gzplugin_joint_control robot_components_namespace="$(arg robot_components_namespace)"
-                                  trajectory_param_namespace="$(arg trajectory_param_namespace)"/>
+        <xacro:gzplugin_joint_control robot_components_namespace="$(arg robot_components_namespace)" trajectory_param_namespace="$(arg trajectory_param_namespace)"/>
   </xacro:unless>
   <xacro:if value="$(arg load_grasp_fix)">
